Commit message: feat(rby1_description): align URDF with rby1-sdk
- Rename links to match SDK: base, link_torso_N, link_right/left_arm_N,
  link_head_N, wheel_r, wheel_l, wheel_fr/fl/rr/rl_link,
  FT_sensor_R/L, ee_right/left, ee_finger_r1/r2/l1/l2
- Update joint axes, origins, and limits to match SDK exactly
- Add FT sensor, end-effector, and head_base fixed joints
- Replace box geometry with real .dae mesh files from rby1-sdk
- Add meshes/ directories: rby1a (38 files), rby1m (47 files)
- Parameterize macros with model and torso_0_xyz arguments
- Update CMakeLists.txt to install meshes directory

File: rby1_description/urdf/rby1.common.xacro (robot description, xacro)
@@ -1,104 +1,807 @@
 <?xml version="1.0"?>
 <robot xmlns:xacro="http://www.ros.org/wiki/xacro">
-  <material name="rby1_dark">
-    <color rgba="0.08 0.09 0.10 1.0"/>
-  </material>
-  <material name="rby1_light">
-    <color rgba="0.72 0.74 0.76 1.0"/>
-  </material>
-  <xacro:macro name="simple_box_link" params="name size color">
-    <link name="${name}">
-      <visual>
-        <geometry>
-          <box size="${size}"/>
-        </geometry>
-        <material name="${color}"/>
-      </visual>
-      <collision>
-        <geometry>
-          <box size="${size}"/>
-        </geometry>
-      </collision>
-    </link>
+  <!-- ============================================================
+       rby1_upper_body: torso + arms + head + FT sensors + EE
+       params:
+         model        - "rby1a" or "rby1m" (selects mesh subdirectory)
+         torso_0_xyz  - origin xyz of torso_0 joint (differs per platform)
+  ============================================================ -->
+  <xacro:macro name="rby1_upper_body" params="model torso_0_xyz">
+    <!-- Torso links -->
+    <link name="link_torso_0">
+      <inertial>
+        <mass value="2.24282123"/>
+        <origin rpy="0 0 0" xyz="-0.08848415 0.00021367 0.00000046"/>
+        <inertia ixx="0.01413496" ixy="0.00092982" ixz="-0.00000010"
+                 iyy="0.01005357" iyz="-0.00000008" izz="0.01892525"/>
+      </inertial>
+      <visual>
+        <geometry>
+          <mesh filename="package://rby1_description/meshes/${model}/LINK_1.dae"/>
+        </geometry>
+      </visual>
+    </link>
+    <link name="link_torso_1">
+      <inertial>
+        <mass value="9.72162676"/>
+        <origin rpy="0 0 0" xyz="0.00728955 -0.01728522 0.06911380"/>
+        <inertia ixx="0.14862640" ixy="-0.00142621" ixz="-0.00951385"
+                 iyy="0.13854733" iyz="-0.00975351" izz="0.02912982"/>
+      </inertial>
+      <visual>
+        <geometry>
+          <mesh filename="package://rby1_description/meshes/${model}/LINK_2.dae"/>
+        </geometry>
+      </visual>
+    </link>
+    <link name="link_torso_2">
+      <inertial>
+        <mass value="9.21691850"/>
+        <origin rpy="0 0 0" xyz="0.00653835 -0.01769536 0.05636582"/>
+        <inertia ixx="0.12162270" ixy="-0.00127910" ixz="-0.00831678"
+                 iyy="0.11589190" iyz="-0.00873271" izz="0.03094484"/>
+      </inertial>
+      <visual>
+        <geometry>
+          <mesh filename="package://rby1_description/meshes/${model}/LINK_3.dae"/>
+        </geometry>
+      </visual>
+    </link>
+    <link name="link_torso_3">
+      <inertial>
+        <mass value="4.18679196"/>
+        <origin rpy="0 0 0" xyz="-0.00574156 -0.01725975 0.00005610"/>
+        <inertia ixx="0.00849870" ixy="0.00040861" ixz="-0.00000263"
+                 iyy="0.00929513" iyz="-0.00001243" izz="0.00955442"/>
+      </inertial>
+      <visual>
+        <geometry>
+          <mesh filename="package://rby1_description/meshes/${model}/LINK_4.dae"/>
+        </geometry>
+      </visual>
+    </link>
+    <link name="link_torso_4">
+      <inertial>
+        <mass value="4.45566276"/>
+        <origin rpy="0 0 0" xyz="-0.09097095 0.00005085 0.02601950"/>
+        <inertia ixx="0.01545991" ixy="0.00001883" ixz="-0.00780349"
+                 iyy="0.02550888" iyz="0.00000715" izz="0.01952563"/>
+      </inertial>
+      <visual>
+        <geometry>
+          <mesh filename="package://rby1_description/meshes/${model}/LINK_5.dae"/>
+        </geometry>
+      </visual>
+    </link>
+    <link name="link_torso_5">
+      <inertial>
+        <mass value="12.59012341"/>
+        <origin rpy="0 0 0" xyz="-0.01338376 0.00025621 -0.03272487"/>
+        <inertia ixx="0.21375525" ixy="0.00051520" ixz="0.00880124"
+                 iyy="0.16562090" iyz="-0.00023995" izz="0.13308879"/>
+      </inertial>
+      <visual>
+        <geometry>
+          <mesh filename="package://rby1_description/meshes/${model}/LINK_6.dae"/>
+        </geometry>
+      </visual>
+    </link>
+    <!-- Right arm links -->
+    <link name="link_right_arm_0">
+      <inertial>
+        <mass value="1.26164242"/>
+        <origin rpy="0 0 0" xyz="-0.00316662 0.03437181 -0.00000030"/>
+        <inertia ixx="0.00230621" ixy="0.00039024" ixz="-0.00000256"
+                 iyy="0.00426418" iyz="0.00000118" izz="0.00432156"/>
+      </inertial>
+      <visual>
+        <geometry>
+          <mesh filename="package://rby1_description/meshes/${model}/LINK_7.dae"/>
+        </geometry>
+      </visual>
+    </link>
+    <link name="link_right_arm_1">
+      <inertial>
+        <mass value="2.27287031"/>
+        <origin rpy="0 0 0" xyz="-0.00307855 -0.00124741 -0.01294324"/>
+        <inertia ixx="0.00388490" ixy="-0.00001477" ixz="0.00011465"
+                 iyy="0.00447034" iyz="-0.00010023" izz="0.00288341"/>
+      </inertial>
+      <visual>
+        <geometry>
+          <mesh filename="package://rby1_description/meshes/${model}/LINK_8.dae"/>
+        </geometry>
+      </visual>
+    </link>
+    <link name="link_right_arm_2">
+      <inertial>
+        <mass value="2.46909439"/>
+        <origin rpy="0 0 0" xyz="0.00115434 0.00196635 -0.16192524"/>
+        <inertia ixx="0.00980269" ixy="0.00005871" ixz="0.00051888"
+                 iyy="0.00924560" iyz="-0.00045932" izz="0.00329867"/>
+      </inertial>
+      <visual>
+        <geometry>
+          <mesh filename="package://rby1_description/meshes/${model}/LINK_9.dae"/>
+        </geometry>
+      </visual>
+    </link>
+    <link name="link_right_arm_3">
+      <inertial>
+        <mass value="2.26099493"/>
+        <origin rpy="0 0 0" xyz="-0.01603135 -0.00692891 -0.04549811"/>
+        <inertia ixx="0.00822606" ixy="0.00027620" ixz="-0.00156570"
+                 iyy="0.00844870" iyz="0.00076157" izz="0.00236614"/>
+      </inertial>
+      <visual>
+        <geometry>
+          <mesh filename="package://rby1_description/meshes/${model}/LINK_10.dae"/>
+        </geometry>
+      </visual>
+    </link>
+    <link name="link_right_arm_4">
+      <inertial>
+        <mass value="0.42508710"/>
+        <origin rpy="0 0 0" xyz="-0.00000011 -0.02696036 0.06182110"/>
+        <inertia ixx="0.00082466" ixy="0.0" ixz="0.0"
+                 iyy="0.00075398" iyz="-0.00025338" izz="0.00039794"/>
+      </inertial>
+      <visual>
+        <geometry>
+          <mesh filename="package://rby1_description/meshes/${model}/LINK_11.dae"/>
+        </geometry>
+      </visual>
+    </link>
+    <link name="link_right_arm_5">
+      <inertial>
+        <mass value="1.59194395"/>
+        <origin rpy="0 0 0" xyz="0.00318034 -0.00532264 -0.02809655"/>
+        <inertia ixx="0.00256054" ixy="-0.00002344" ixz="-0.00001563"
+                 iyy="0.00257233" iyz="0.00021608" izz="0.00156092"/>
+      </inertial>
+      <visual>
+        <geometry>
+          <mesh filename="package://rby1_description/meshes/${model}/LINK_12.dae"/>
+        </geometry>
+      </visual>
+    </link>
+    <link name="link_right_arm_6">
+      <inertial>
+        <mass value="0.21137279"/>
+        <origin rpy="0 0 0" xyz="0.00066810 -0.00031708 -0.09636043"/>
+        <inertia ixx="0.00013511" ixy="-0.00000242" ixz="-0.00000102"
+                 iyy="0.00014453" iyz="0.00000094" izz="0.00025431"/>
+      </inertial>
+      <visual>
+        <geometry>
+          <mesh filename="package://rby1_description/meshes/${model}/LINK_13.dae"/>
+        </geometry>
+      </visual>
+    </link>
+    <!-- Left arm links -->
+    <link name="link_left_arm_0">
+      <inertial>
+        <mass value="1.26164242"/>
+        <origin rpy="0 0 0" xyz="-0.00316662 -0.03437181 -0.00000030"/>
+        <inertia ixx="0.00230621" ixy="-0.00039024" ixz="0.00000256"
+                 iyy="0.00426418" iyz="0.00000118" izz="0.00432156"/>
+      </inertial>
+      <visual>
+        <geometry>
+          <mesh filename="package://rby1_description/meshes/${model}/LINK_14.dae"/>
+        </geometry>
+      </visual>
+    </link>
+    <link name="link_left_arm_1">
+      <inertial>
+        <mass value="2.27287031"/>
+        <origin rpy="0 0 0" xyz="-0.00307855 0.00124741 -0.01294324"/>
+        <inertia ixx="0.00388490" ixy="-0.00001477" ixz="0.00011465"
+                 iyy="0.00447034" iyz="0.00010023" izz="0.00288341"/>
+      </inertial>
+      <visual>
+        <geometry>
+          <mesh filename="package://rby1_description/meshes/${model}/LINK_15.dae"/>
+        </geometry>
+      </visual>
+    </link>
+    <link name="link_left_arm_2">
+      <inertial>
+        <mass value="2.46909439"/>
+        <origin rpy="0 0 0" xyz="0.00115434 -0.00196635 -0.16192524"/>
+        <inertia ixx="0.00980269" ixy="0.00005871" ixz="0.00051888"
+                 iyy="0.00924560" iyz="-0.00045932" izz="0.00329867"/>
+      </inertial>
+      <visual>
+        <geometry>
+          <mesh filename="package://rby1_description/meshes/${model}/LINK_16.dae"/>
+        </geometry>
+      </visual>
+    </link>
+    <link name="link_left_arm_3">
+      <inertial>
+        <mass value="2.26099493"/>
+        <origin rpy="0 0 0" xyz="-0.01603135 0.00692891 -0.04549811"/>
+        <inertia ixx="0.00822606" ixy="-0.00027620" ixz="-0.00156570"
+                 iyy="0.00844870" iyz="-0.00076157" izz="0.00236614"/>
+      </inertial>
+      <visual>
+        <geometry>
+          <mesh filename="package://rby1_description/meshes/${model}/LINK_17.dae"/>
+        </geometry>
+      </visual>
+    </link>
+    <link name="link_left_arm_4">
+      <inertial>
+        <mass value="0.42508710"/>
+        <origin rpy="0 0 0" xyz="0.00000011 0.02696036 0.06182110"/>
+        <inertia ixx="0.00082466" ixy="0.0" ixz="0.0"
+                 iyy="0.00075398" iyz="0.00025338" izz="0.00039794"/>
+      </inertial>
+      <visual>
+        <geometry>
+          <mesh filename="package://rby1_description/meshes/${model}/LINK_18.dae"/>
+        </geometry>
+      </visual>
+    </link>
+    <link name="link_left_arm_5">
+      <inertial>
+        <mass value="1.59194395"/>
+        <origin rpy="0 0 0" xyz="0.00318034 0.00532264 -0.02809655"/>
+        <inertia ixx="0.00256054" ixy="0.00002344" ixz="-0.00001563"
+                 iyy="0.00257233" iyz="-0.00021608" izz="0.00156092"/>
+      </inertial>
+      <visual>
+        <geometry>
+          <mesh filename="package://rby1_description/meshes/${model}/LINK_19.dae"/>
+        </geometry>
+      </visual>
+    </link>
+    <link name="link_left_arm_6">
+      <inertial>
+        <mass value="0.21137279"/>
+        <origin rpy="0 0 0" xyz="-0.00066810 0.00031708 -0.09636043"/>
+        <inertia ixx="0.00013511" ixy="-0.00000242" ixz="0.00000102"
+                 iyy="0.00014453" iyz="-0.00000094" izz="0.00025431"/>
+      </inertial>
+      <visual>
+        <geometry>
+          <mesh filename="package://rby1_description/meshes/${model}/LINK_20.dae"/>
+        </geometry>
+      </visual>
+    </link>
+    <!-- FT sensors -->
+    <link name="FT_sensor_R">
+      <inertial>
+        <mass value="0.49078507"/>
+        <origin rpy="0 0 0" xyz="0.00010423 0.00108019 -0.01880676"/>
+        <inertia ixx="0.00028587" ixy="-0.00000146" ixz="-0.00000026"
+                 iyy="0.00030459" iyz="-0.00000772" izz="0.00036377"/>
+      </inertial>
+      <visual>
+        <geometry>
+          <mesh filename="package://rby1_description/meshes/${model}/FT_SENSOR_R.dae"/>
+        </geometry>
+      </visual>
+    </link>
+    <link name="FT_sensor_L">
+      <inertial>
+        <mass value="0.49078507"/>
+        <origin rpy="0 0 0" xyz="-0.00010423 -0.00108019 -0.01880676"/>
+        <inertia ixx="0.00028587" ixy="-0.00000146" ixz="0.00000026"
+                 iyy="0.00030459" iyz="0.00000772" izz="0.00036377"/>
+      </inertial>
+      <visual>
+        <geometry>
+          <mesh filename="package://rby1_description/meshes/${model}/FT_SENSOR_L.dae"/>
+        </geometry>
+      </visual>
+    </link>
+    <!-- End effectors (right) -->
+    <link name="ee_right">
+      <inertial>
+        <mass value="0.46704998"/>
+        <origin rpy="0 0 0" xyz="0.00212703 0.00000615 -0.04287176"/>
+        <inertia ixx="0.00032067" ixy="0.00002383" ixz="-0.00000785"
+                 iyy="0.00059559" iyz="-0.00000007" izz="0.00052732"/>
+      </inertial>
+      <visual>
+        <geometry>
+          <mesh filename="package://rby1_description/meshes/${model}/EE_BODY.dae"/>
+        </geometry>
+      </visual>
+    </link>
+    <link name="ee_finger_r1">
+      <inertial>
+        <mass value="0.03326999"/>
+        <origin rpy="0 0 0" xyz="0.00278346 -0.00000329 -0.02570112"/>
+        <inertia ixx="0.00001231" ixy="0.0" ixz="-0.00000042"
+                 iyy="0.00001066" iyz="0.0" izz="0.00000224"/>
+      </inertial>
+      <visual>
+        <geometry>
+          <mesh filename="package://rby1_description/meshes/${model}/EE_FINGER.dae"/>
+        </geometry>
+      </visual>
+    </link>
+    <link name="ee_finger_r2">
+      <inertial>
+        <mass value="0.03326999"/>
+        <origin rpy="0 0 0" xyz="0.00278346 -0.00000329 -0.02570112"/>
+        <inertia ixx="0.00001231" ixy="0.0" ixz="-0.00000042"
+                 iyy="0.00001066" iyz="0.0" izz="0.00000224"/>
+      </inertial>
+      <visual>
+        <geometry>
+          <mesh filename="package://rby1_description/meshes/${model}/EE_FINGER.dae"/>
+        </geometry>
+      </visual>
+    </link>
+    <!-- End effectors (left) -->
+    <link name="ee_left">
+      <inertial>
+        <mass value="0.46704998"/>
+        <origin rpy="0 0 0" xyz="0.00212703 0.00000615 -0.04287176"/>
+        <inertia ixx="0.00032067" ixy="0.00002383" ixz="-0.00000785"
+                 iyy="0.00059559" iyz="-0.00000007" izz="0.00052732"/>
+      </inertial>
+      <visual>
+        <geometry>
+          <mesh filename="package://rby1_description/meshes/${model}/EE_BODY.dae"/>
+        </geometry>
+      </visual>
+    </link>
+    <link name="ee_finger_l1">
+      <inertial>
+        <mass value="0.03326999"/>
+        <origin rpy="0 0 0" xyz="0.00278346 -0.00000329 -0.02570112"/>
+        <inertia ixx="0.00001231" ixy="0.0" ixz="-0.00000042"
+                 iyy="0.00001066" iyz="0.0" izz="0.00000224"/>
+      </inertial>
+      <visual>
+        <geometry>
+          <mesh filename="package://rby1_description/meshes/${model}/EE_FINGER.dae"/>
+        </geometry>
+      </visual>
+    </link>
+    <link name="ee_finger_l2">
+      <inertial>
+        <mass value="0.03326999"/>
+        <origin rpy="0 0 0" xyz="0.00278346 -0.00000329 -0.02570112"/>
+        <inertia ixx="0.00001231" ixy="0.0" ixz="-0.00000042"
+                 iyy="0.00001066" iyz="0.0" izz="0.00000224"/>
+      </inertial>
+      <visual>
+        <geometry>
+          <mesh filename="package://rby1_description/meshes/${model}/EE_FINGER.dae"/>
+        </geometry>
+      </visual>
+    </link>
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
File: rby1_description/urdf/rby1a.urdf.xacro (robot description, xacro)
@@ -8,6 +8,6 @@
   <xacro:include filename="$(find rby1_description)/urdf/rby1.common.xacro"/>
   <xacro:include filename="$(find rby1_description)/urdf/rby1.ros2_control.xacro"/>
-  <xacro:rby1_upper_body/>
-  <xacro:rby1a_mobility/>
+  <xacro:rby1a_mobility model="rby1a"/>
+  <xacro:rby1_upper_body model="rby1a" torso_0_xyz="0 0 0.2805"/>
   <xacro:rby1a_ros2_control
     robot_ip="$(arg robot_ip)"

File: rby1_description/urdf/rby1m.urdf.xacro (robot description, xacro)
@@ -8,6 +8,6 @@
   <xacro:include filename="$(find rby1_description)/urdf/rby1.common.xacro"/>
   <xacro:include filename="$(find rby1_description)/urdf/rby1.ros2_control.xacro"/>
-  <xacro:rby1_upper_body/>
-  <xacro:rby1m_mobility/>
+  <xacro:rby1m_mobility model="rby1m"/>
+  <xacro:rby1_upper_body model="rby1m" torso_0_xyz="0 0 0.2965"/>
   <xacro:rby1m_ros2_control
     robot_ip="$(arg robot_ip)"
