Commit message: feat(rby1_description): support all models and versions (rby1a/m v1.0-v1.3, rby1ub)
- Vendor SDK URDFs as xacros for each model/version:
  rby1a: v1.0, v1.1, v1.2
  rby1m: v1.0, v1.1, v1.2, v1.3 (v1.3 adds WY/WP/WR wrist links)
  rby1ub: single variant (upper-body only, no mobility)

- Transformations applied during vendoring:
  - Mesh paths rewritten to package://rby1_description/meshes/<model>/
  - xacro namespace added to root <robot> element
  - SDK-specific <mobile/> elements removed (not valid URDF)
  - Non-standard in_model_type attributes removed
  - <capsule> collision geometry converted to <cylinder> (same R/L)
  - Missing effort attribute added to continuous-joint <limit> elements

- rby1a.urdf.xacro, rby1m.urdf.xacro: rewritten as thin wrappers;
  accept new 'version' arg (default: 1.2); rby1.common.xacro deleted

- rby1ub.urdf.xacro: new top-level wrapper for the upper-body platform

- rby1.ros2_control.xacro: add rby1ub_ros2_control macro
  (joints: torso_hp, torso_5, arm x14, head x2)

- meshes/rby1ub/: add 24 DAE meshes vendored from rby1-sdk

- Launch files updated (rby1_description and rby1_bringup):
  - model arg extended to accept 'a', 'm', or 'ub'
  - version arg added (default: 1.2; ignored for ub)

All 8 combinations (a-1.0/1.1/1.2, m-1.0/1.1/1.2/1.3, ub) validated
with check_urdf.

File: rby1_description/urdf/rby1.ros2_control.xacro (robot description, xacro)
@@ -101,3 +101,32 @@
     </ros2_control>
   </xacro:macro>
+  <xacro:macro name="rby1ub_ros2_control" params="robot_ip use_mock_hardware auto_reconnect read_timeout_sec connect_timeout_sec">
+    <ros2_control name="RBY1System" type="system">
+      <xacro:rby1_hardware_block
+        robot_ip="${robot_ip}"
+        model="ub"
+        use_mock_hardware="${use_mock_hardware}"
+        auto_reconnect="${auto_reconnect}"
+        read_timeout_sec="${read_timeout_sec}"
+        connect_timeout_sec="${connect_timeout_sec}"/>
+      <xacro:rby1_state_interfaces joint_name="torso_hp"/>
+      <xacro:rby1_state_interfaces joint_name="torso_5"/>
+      <xacro:rby1_state_interfaces joint_name="right_arm_0"/>
+      <xacro:rby1_state_interfaces joint_name="right_arm_1"/>
+      <xacro:rby1_state_interfaces joint_name="right_arm_2"/>
+      <xacro:rby1_state_interfaces joint_name="right_arm_3"/>
+      <xacro:rby1_state_interfaces joint_name="right_arm_4"/>
+      <xacro:rby1_state_interfaces joint_name="right_arm_5"/>
+      <xacro:rby1_state_interfaces joint_name="right_arm_6"/>
+      <xacro:rby1_state_interfaces joint_name="left_arm_0"/>
+      <xacro:rby1_state_interfaces joint_name="left_arm_1"/>
+      <xacro:rby1_state_interfaces joint_name="left_arm_2"/>
+      <xacro:rby1_state_interfaces joint_name="left_arm_3"/>
+      <xacro:rby1_state_interfaces joint_name="left_arm_4"/>
+      <xacro:rby1_state_interfaces joint_name="left_arm_5"/>
+      <xacro:rby1_state_interfaces joint_name="left_arm_6"/>
+      <xacro:rby1_state_interfaces joint_name="head_0"/>
+      <xacro:rby1_state_interfaces joint_name="head_1"/>
+    </ros2_control>
+  </xacro:macro>
 </robot>

File: rby1_description/urdf/rby1a.urdf.xacro (robot description, xacro)
@@ -1,4 +1,10 @@
 <?xml version="1.0"?>
 <robot name="rby1a" xmlns:xacro="http://www.ros.org/wiki/xacro">
+  <!--
+    Top-level wrapper for the RBY1-A platform.
+    Supported versions: 1.0, 1.1, 1.2 (default).
+    Vendored from rby1-sdk/models/rby1a/urdf/model_v<version>.urdf.
+  -->
+  <xacro:arg name="version" default="1.2"/>
   <xacro:arg name="robot_ip" default="127.0.0.1:50051"/>
   <xacro:arg name="use_mock_hardware" default="false"/>
@@ -6,8 +12,6 @@
   <xacro:arg name="read_timeout_sec" default="0.5"/>
   <xacro:arg name="connect_timeout_sec" default="3.0"/>
-  <xacro:include filename="$(find rby1_description)/urdf/rby1.common.xacro"/>
+  <xacro:include filename="$(find rby1_description)/urdf/rby1a/v$(arg version)/model.xacro"/>
   <xacro:include filename="$(find rby1_description)/urdf/rby1.ros2_control.xacro"/>
-  <xacro:rby1a_mobility model="rby1a"/>
-  <xacro:rby1_upper_body model="rby1a" torso_0_xyz="0 0 0.2805"/>
   <xacro:rby1a_ros2_control
     robot_ip="$(arg robot_ip)"

File: rby1_description/urdf/rby1ub.urdf.xacro (robot description, xacro)
@@ -1,18 +1,16 @@
 <?xml version="1.0"?>
-<robot name="rby1m" xmlns:xacro="http://www.ros.org/wiki/xacro">
+<robot name="rby1ub" xmlns:xacro="http://www.ros.org/wiki/xacro">
   <!--
-    Top-level wrapper for the RBY1-M platform.
-    Supported versions: 1.0, 1.1, 1.2 (default), 1.3 (WY/WP/WR wrist).
-    Vendored from rby1-sdk/models/rby1m/urdf/model_v<version>.urdf.
+    Top-level wrapper for the RBY1 upper-body (UB) platform.
+    Single variant; vendored from rby1-sdk/models/rby1ub/urdf/model.urdf.
   -->
-  <xacro:arg name="version" default="1.2"/>
   <xacro:arg name="robot_ip" default="127.0.0.1:50051"/>
-  <xacro:arg name="use_mock_hardware" default="false"/>
+  <xacro:arg name="use_mock_hardware" default="true"/>
   <xacro:arg name="auto_reconnect" default="true"/>
   <xacro:arg name="read_timeout_sec" default="0.5"/>
   <xacro:arg name="connect_timeout_sec" default="3.0"/>
-  <xacro:include filename="$(find rby1_description)/urdf/rby1m/v$(arg version)/model.xacro"/>
+  <xacro:include filename="$(find rby1_description)/urdf/rby1ub/model.xacro"/>
   <xacro:include filename="$(find rby1_description)/urdf/rby1.ros2_control.xacro"/>
-  <xacro:rby1m_ros2_control
+  <xacro:rby1ub_ros2_control
     robot_ip="$(arg robot_ip)"
     use_mock_hardware="$(arg use_mock_hardware)"
