Commit message: update files

File: rby1_moveit_test/config/rby1.ros2_control.xacro (robot description, xacro)
@@ -1,10 +1,18 @@
 <?xml version="1.0"?>
 <robot xmlns:xacro="http://www.ros.org/wiki/xacro">
-    <xacro:macro name="rby1_ros2_control" params="name initial_positions_file">
+    <xacro:macro name="rby1_ros2_control" params="name initial_positions_file use_fake_hardware:=true robot_ip:=127.0.0.1:50051 model:=m collision_check_enable:=false collision_threshold:=0.01">
         <xacro:property name="initial_positions" value="${load_yaml(initial_positions_file)['initial_positions']}"/>
         <ros2_control name="${name}" type="system">
             <hardware>
-                <!-- By default, set up controllers for simulation. This won't work on real hardware -->
-                <plugin>mock_components/GenericSystem</plugin>
+                <xacro:if value="${use_fake_hardware}">
+                    <plugin>mock_components/GenericSystem</plugin>
+                </xacro:if>
+                <xacro:unless value="${use_fake_hardware}">
+                    <plugin>rby1_hardware/RBY1SystemHardware</plugin>
+                    <param name="robot_ip">${robot_ip}</param>
+                    <param name="model">${model}</param>
+                    <param name="collision_check_enable">${collision_check_enable}</param>
+                    <param name="collision_threshold">${collision_threshold}</param>
+                </xacro:unless>
             </hardware>
             <joint name="left_arm_0">

File: rby1_moveit_test/config/rby1.urdf.xacro (robot description, xacro)
@@ -2,8 +2,23 @@
 <robot xmlns:xacro="http://www.ros.org/wiki/xacro" name="rby1">
     <xacro:arg name="initial_positions_file" default="initial_positions.yaml" />
+    <xacro:arg name="use_fake_hardware" default="true" />
+    <xacro:arg name="robot_ip" default="127.0.0.1:50051" />
+    <xacro:arg name="model" default="m" />
+    <xacro:arg name="collision_check_enable" default="false" />
+    <xacro:arg name="collision_threshold" default="0.01" />
+    <xacro:arg name="model_name" default="rby1m" />
+    <xacro:arg name="model_version" default="1_3" />
     <!-- Import rby1 urdf file -->
-    <xacro:include filename="$(find rby1_description)/urdf/rby1.urdf" />
+    <xacro:include filename="$(find rby1_description)/urdf/$(arg model_name)/model_v$(arg model_version).urdf" />
     <!-- Import control_xacro -->
     <xacro:include filename="rby1.ros2_control.xacro" />
-    <xacro:rby1_ros2_control name="FakeSystem" initial_positions_file="$(arg initial_positions_file)"/>
+    <xacro:rby1_ros2_control
+        name="RBY1System"
+        initial_positions_file="$(arg initial_positions_file)"
+        use_fake_hardware="$(arg use_fake_hardware)"
+        robot_ip="$(arg robot_ip)"
+        model="$(arg model)"
+        collision_check_enable="$(arg collision_check_enable)"
+        collision_threshold="$(arg collision_threshold)"
+    />
 </robot>

Commit message: add moveit_m_1_2 package

File: rby1_moveit_test/config/rby1.ros2_control.xacro (robot description, xacro)
@@ -2,5 +2,5 @@
 <robot xmlns:xacro="http://www.ros.org/wiki/xacro">
     <xacro:macro name="rby1_ros2_control" params="name initial_positions_file use_fake_hardware:=true robot_ip:=127.0.0.1:50051 model:=m collision_check_enable:=false collision_threshold:=0.01">
-        <xacro:property name="initial_positions" value="${load_yaml(initial_positions_file)['initial_positions']}"/>
+        <xacro:property name="initial_positions" value="${xacro.load_yaml(initial_positions_file)['initial_positions']}"/>
         <ros2_control name="${name}" type="system">
             <hardware>
