Commit message: update files

File: rby1_description/urdf/rby1a/model_v1_1.urdf (robot description, URDF)
Before this commit: robot RBY1_A_v1_1, 34 links, 33 joints
Links:
- removed link ee_finger_l1
- removed link ee_finger_l2
- removed link ee_finger_r1
- removed link ee_finger_r2
- removed link ee_virtual_left
- removed link ee_virtual_right
- added link gripper_finger_l1, mass 0.03326999; collision mesh filename=package://rby1_description/meshes/rby1a/EE_FINGER.dae; visual mesh filename=package://rby1_description/meshes/rby1a/EE_FINGER.dae
- added link gripper_finger_l2, mass 0.03326999; collision mesh filename=package://rby1_description/meshes/rby1a/EE_FINGER.dae; visual mesh filename=package://rby1_description/meshes/rby1a/EE_FINGER.dae
- added link gripper_finger_r1, mass 0.03326999; collision mesh filename=package://rby1_description/meshes/rby1a/EE_FINGER.dae; visual mesh filename=package://rby1_description/meshes/rby1a/EE_FINGER.dae
- added link gripper_finger_r2, mass 0.03326999; collision mesh filename=package://rby1_description/meshes/rby1a/EE_FINGER.dae; visual mesh filename=package://rby1_description/meshes/rby1a/EE_FINGER.dae
- added link gripper_left, mass 0.46704998; collision mesh filename=package://rby1_description/meshes/rby1a/EE_BODY.dae; visual mesh filename=package://rby1_description/meshes/rby1a/EE_BODY.dae
- added link gripper_right, mass 0.46704998; collision mesh filename=package://rby1_description/meshes/rby1a/EE_BODY.dae; visual mesh filename=package://rby1_description/meshes/rby1a/EE_BODY.dae
- link ee_left: mass 0.46704998 -> None; geometry 
- link ee_right: mass 0.46704998 -> None; geometry 
Joints:
- removed joint end_effector_left
- removed joint end_effector_right
- removed joint gripper_finger_l1
- removed joint gripper_finger_l2
- removed joint gripper_finger_r1
- removed joint gripper_finger_r2
- removed joint tool_left
- removed joint tool_right
- added joint ee_left_joint: type fixed, parent link_left_arm_6, child ee_left, origin xyz=0.0 0.0 -0.1261 rpy=0 0.0 0.0, axis 0 0 1
- added joint ee_right_joint: type fixed, parent link_right_arm_6, child ee_right, origin xyz=0.0 0.0 -0.1261 rpy=0 0.0 0.0, axis 0 0 1
- added joint gripper_finger_l1_joint: type prismatic, parent gripper_left, child gripper_finger_l1, origin xyz=0.003 0.0 -0.075 rpy=0.0 0.0 0.0, axis -1 0 0, limit lower=-0.05 upper=0 effort=1000 velocity=0.05
- added joint gripper_finger_l2_joint: type prismatic, parent gripper_left, child gripper_finger_l2, origin xyz=-0.003 0.0 -0.075 rpy=0.0 0.0 3.1415926535, axis 1 0 0, limit lower=0 upper=0.05 effort=1000 velocity=0.05, mimic joint=gripper_finger_l1_joint multiplier=1.0 offset=0.0
- added joint gripper_finger_r1_joint: type prismatic, parent gripper_right, child gripper_finger_r1, origin xyz=0.003 0.0 -0.075 rpy=0.0 0.0 0.0, axis -1 0 0, limit lower=-0.05 upper=0 effort=1000 velocity=0.05
- added joint gripper_finger_r2_joint: type prismatic, parent gripper_right, child gripper_finger_r2, origin xyz=-0.003 0.0 -0.075 rpy=0.0 0.0 3.1415926535, axis 1 0 0, limit lower=0 upper=0.05 effort=1000 velocity=0.05, mimic joint=gripper_finger_r1_joint multiplier=1.0 offset=0.0
- added joint gripper_left_joint: type fixed, parent ee_left, child gripper_left, origin xyz=0.0 0.0 0.0 rpy=0 0.0 0.0, axis 0 0 0
- added joint gripper_right_joint: type fixed, parent ee_right, child gripper_right, origin xyz=0.0 0.0 0.0 rpy=0 0.0 0.0, axis 0 0 0

File: rby1_description/urdf/rby1a/model_v1_2.urdf (robot description, URDF)
Before this commit: robot RBY1_A_v1_2, 34 links, 33 joints
Links:
- removed link ee_finger_l1
- removed link ee_finger_l2
- removed link ee_finger_r1
- removed link ee_finger_r2
- removed link ee_virtual_left
- removed link ee_virtual_right
- added link gripper_finger_l1, mass 0.03326999; collision mesh filename=package://rby1_description/meshes/rby1a/EE_FINGER.dae; visual mesh filename=package://rby1_description/meshes/rby1a/EE_FINGER.dae
- added link gripper_finger_l2, mass 0.03326999; collision mesh filename=package://rby1_description/meshes/rby1a/EE_FINGER.dae; visual mesh filename=package://rby1_description/meshes/rby1a/EE_FINGER.dae
- added link gripper_finger_r1, mass 0.03326999; collision mesh filename=package://rby1_description/meshes/rby1a/EE_FINGER.dae; visual mesh filename=package://rby1_description/meshes/rby1a/EE_FINGER.dae
- added link gripper_finger_r2, mass 0.03326999; collision mesh filename=package://rby1_description/meshes/rby1a/EE_FINGER.dae; visual mesh filename=package://rby1_description/meshes/rby1a/EE_FINGER.dae
- added link gripper_left, mass 0.46704998; collision mesh filename=package://rby1_description/meshes/rby1a/EE_BODY.dae; visual mesh filename=package://rby1_description/meshes/rby1a/EE_BODY.dae
- added link gripper_right, mass 0.46704998; collision mesh filename=package://rby1_description/meshes/rby1a/EE_BODY.dae; visual mesh filename=package://rby1_description/meshes/rby1a/EE_BODY.dae
- link ee_left: mass 0.46704998 -> None; geometry 
- link ee_right: mass 0.46704998 -> None; geometry 
Joints:
- removed joint end_effector_left
- removed joint end_effector_right
- removed joint gripper_finger_l1
- removed joint gripper_finger_l2
- removed joint gripper_finger_r1
- removed joint gripper_finger_r2
- removed joint tool_left
- removed joint tool_right
- added joint ee_left_joint: type fixed, parent link_left_arm_6, child ee_left, origin xyz=0.0 0.0 -0.1261 rpy=0 0.0 0.0, axis 0 0 1
- added joint ee_right_joint: type fixed, parent link_right_arm_6, child ee_right, origin xyz=0.0 0.0 -0.1261 rpy=0 0.0 0.0, axis 0 0 1
- added joint gripper_finger_l1_joint: type prismatic, parent gripper_left, child gripper_finger_l1, origin xyz=0.003 0.0 -0.075 rpy=0.0 0.0 0.0, axis -1 0 0, limit lower=-0.05 upper=0 effort=1000 velocity=0.05
- added joint gripper_finger_l2_joint: type prismatic, parent gripper_left, child gripper_finger_l2, origin xyz=-0.003 0.0 -0.075 rpy=0.0 0.0 3.1415926535, axis 1 0 0, limit lower=0 upper=0.05 effort=1000 velocity=0.05, mimic joint=gripper_finger_l1_joint multiplier=1.0 offset=0.0
- added joint gripper_finger_r1_joint: type prismatic, parent gripper_right, child gripper_finger_r1, origin xyz=0.003 0.0 -0.075 rpy=0.0 0.0 0.0, axis -1 0 0, limit lower=-0.05 upper=0 effort=1000 velocity=0.05
- added joint gripper_finger_r2_joint: type prismatic, parent gripper_right, child gripper_finger_r2, origin xyz=-0.003 0.0 -0.075 rpy=0.0 0.0 3.1415926535, axis 1 0 0, limit lower=0 upper=0.05 effort=1000 velocity=0.05
- added joint gripper_left_joint: type fixed, parent ee_left, child gripper_left, origin xyz=0.0 0.0 0.0 rpy=0 0.0 0.0, axis 0 0 0
- added joint gripper_right_joint: type fixed, parent ee_right, child gripper_right, origin xyz=0.0 0.0 0.0 rpy=0 0.0 0.0, axis 0 0 0

File: rby1_description/urdf/rby1m/model_v1_0.urdf (robot description, URDF)
Before this commit: robot RBY1_M_v1_0, 36 links, 35 joints
Links:
- removed link ee_finger_l1
- removed link ee_finger_l2
- removed link ee_finger_r1
- removed link ee_finger_r2
- added link gripper_finger_l1, mass 0.03326999; collision mesh filename=package://rby1_description/meshes/rby1a/EE_FINGER.dae; visual mesh filename=package://rby1_description/meshes/rby1a/EE_FINGER.dae
- added link gripper_finger_l2, mass 0.03326999; collision mesh filename=package://rby1_description/meshes/rby1a/EE_FINGER.dae; visual mesh filename=package://rby1_description/meshes/rby1a/EE_FINGER.dae
- added link gripper_finger_r1, mass 0.03326999; collision mesh filename=package://rby1_description/meshes/rby1a/EE_FINGER.dae; visual mesh filename=package://rby1_description/meshes/rby1a/EE_FINGER.dae
- added link gripper_finger_r2, mass 0.03326999; collision mesh filename=package://rby1_description/meshes/rby1a/EE_FINGER.dae; visual mesh filename=package://rby1_description/meshes/rby1a/EE_FINGER.dae
- added link gripper_left, mass 0.46704998; collision mesh filename=package://rby1_description/meshes/rby1a/EE_BODY.dae; visual mesh filename=package://rby1_description/meshes/rby1a/EE_BODY.dae
- added link gripper_right, mass 0.46704998; collision mesh filename=package://rby1_description/meshes/rby1a/EE_BODY.dae; visual mesh filename=package://rby1_description/meshes/rby1a/EE_BODY.dae
- link ee_left: mass 0.46704998 -> None; geometry 
- link ee_right: mass 0.46704998 -> None; geometry 
Joints:
- removed joint FT_Sensor_END_left
- removed joint FT_Sensor_END_right
- removed joint gripper_finger_l1
- removed joint gripper_finger_l2
- removed joint gripper_finger_r1
- removed joint gripper_finger_r2
- added joint ee_left_joint: type fixed, parent FT_sensor_L, child ee_left, origin xyz=0.0 0.0 0.0 rpy=0.0 0.0 0.0, axis 0 0 1
- added joint ee_right_joint: type fixed, parent FT_sensor_R, child ee_right, origin xyz=0.0 0.0 0.0 rpy=0.0 0.0 0.0, axis 0 0 1
- added joint gripper_finger_l1_joint: type prismatic, parent gripper_left, child gripper_finger_l1, origin xyz=0.003 0.0 -0.073 rpy=0.0 0.0 0.0, axis -1 0 0, limit lower=-0.05 upper=0 effort=1000 velocity=0.05
- added joint gripper_finger_l2_joint: type prismatic, parent gripper_left, child gripper_finger_l2, origin xyz=-0.003 0.0 -0.073 rpy=0.0 0.0 3.1415926535, axis -1 0 0, limit lower=0 upper=0.05 effort=1000 velocity=0.05, mimic joint=gripper_finger_l1_joint multiplier=1.0 offset=0.0
- added joint gripper_finger_r1_joint: type prismatic, parent gripper_right, child gripper_finger_r1, origin xyz=0.003 0.0 -0.073 rpy=0.0 0.0 0.0, axis -1 0 0, limit lower=-0.05 upper=0 effort=1000 velocity=0.05
- added joint gripper_finger_r2_joint: type prismatic, parent gripper_right, child gripper_finger_r2, origin xyz=-0.003 0.0 -0.073 rpy=0.0 0.0 3.1415926535, axis -1 0 0, limit lower=0 upper=0.05 effort=1000 velocity=0.05, mimic joint=gripper_finger_r1_joint multiplier=1.0 offset=0.0
- added joint gripper_left_joint: type fixed, parent ee_left, child gripper_left, origin xyz=0.0 0.0 -0.0461 rpy=0.0 0.0 0.0, axis 0 0 1
- added joint gripper_right_joint: type fixed, parent ee_right, child gripper_right, origin xyz=0.0 0.0 -0.0461 rpy=0.0 0.0 0.0, axis 0 0 1

File: rby1_description/urdf/rby1m/model_v1_1.urdf (robot description, URDF)
Before this commit: robot RBY1_M_v1_1, 34 links, 33 joints
Links:
- removed link ee_finger_l1
- removed link ee_finger_l2
- removed link ee_finger_r1
- removed link ee_finger_r2
- added link gripper_finger_l1, mass 0.03326999; collision mesh filename=package://rby1_description/meshes/rby1m/EE_FINGER.dae; visual mesh filename=package://rby1_description/meshes/rby1m/EE_FINGER.dae
- added link gripper_finger_l2, mass 0.03326999; collision mesh filename=package://rby1_description/meshes/rby1m/EE_FINGER.dae; visual mesh filename=package://rby1_description/meshes/rby1m/EE_FINGER.dae
- added link gripper_finger_r1, mass 0.03326999; collision mesh filename=package://rby1_description/meshes/rby1m/EE_FINGER.dae; visual mesh filename=package://rby1_description/meshes/rby1m/EE_FINGER.dae
- added link gripper_finger_r2, mass 0.03326999; collision mesh filename=package://rby1_description/meshes/rby1m/EE_FINGER.dae; visual mesh filename=package://rby1_description/meshes/rby1m/EE_FINGER.dae
- added link gripper_left, mass 0.46704998; collision mesh filename=package://rby1_description/meshes/rby1m/EE_BODY.dae; visual mesh filename=package://rby1_description/meshes/rby1m/EE_BODY.dae
- added link gripper_right, mass 0.46704998; collision mesh filename=package://rby1_description/meshes/rby1m/EE_BODY.dae; visual mesh filename=package://rby1_description/meshes/rby1m/EE_BODY.dae
- link ee_left: mass 0.46704998 -> None; geometry 
- link ee_right: mass 0.46704998 -> None; geometry 
Joints:
- removed joint gripper_finger_l1
- removed joint gripper_finger_l2
- removed joint gripper_finger_r1
- removed joint gripper_finger_r2
- removed joint tool_left
- removed joint tool_right
- added joint ee_left_joint: type fixed, parent link_left_arm_6, child ee_left, origin xyz=0.0 0.0 -0.1261 rpy=0.0 0.0 0, axis 0 0 1
- added joint ee_right_joint: type fixed, parent link_right_arm_6, child ee_right, origin xyz=0.0 0.0 -0.1261 rpy=0 0.0 0.0, axis 0 0 1
- added joint gripper_finger_l1_joint: type prismatic, parent gripper_left, child gripper_finger_l1, origin xyz=0.003 0.0 -0.075 rpy=0.0 0.0 0.0, axis -1 0 0, limit lower=-0.05 upper=0 effort=1000 velocity=0.05
- added joint gripper_finger_l2_joint: type prismatic, parent gripper_left, child gripper_finger_l2, origin xyz=-0.003 0.0 -0.075 rpy=0.0 0.0 3.1415926535, axis 1 0 0, limit lower=0 upper=0.05 effort=1000 velocity=0.05, mimic joint=gripper_finger_l1_joint multiplier=1.0 offset=0.0
- added joint gripper_finger_r1_joint: type prismatic, parent gripper_right, child gripper_finger_r1, origin xyz=0.003 0.0 -0.075 rpy=0.0 0.0 0.0, axis -1 0 0, limit lower=-0.05 upper=0 effort=1000 velocity=0.05
- added joint gripper_finger_r2_joint: type prismatic, parent gripper_right, child gripper_finger_r2, origin xyz=-0.003 0.0 -0.075 rpy=0.0 0.0 3.1415926535, axis 1 0 0, limit lower=0 upper=0.05 effort=1000 velocity=0.05, mimic joint=gripper_finger_r1_joint multiplier=1.0 offset=0.0
- added joint gripper_left_joint: type fixed, parent ee_left, child gripper_left, origin xyz=0.0 0.0 0.0 rpy=0 0.0 0.0, axis 0 0 0
- added joint gripper_right_joint: type fixed, parent ee_right, child gripper_right, origin xyz=0.0 0.0 0.0 rpy=0 0.0 0.0, axis 0 0 0

File: rby1_description/urdf/rby1m/model_v1_2.urdf (robot description, URDF)
Before this commit: robot RBY1_M_v1_2, 34 links, 33 joints
Links:
- removed link ee_finger_l1
- removed link ee_finger_l2
- removed link ee_finger_r1
- removed link ee_finger_r2
- added link gripper_finger_l1, mass 0.03326999; collision mesh filename=package://rby1_description/meshes/rby1m/EE_FINGER.dae; visual mesh filename=package://rby1_description/meshes/rby1m/EE_FINGER.dae
- added link gripper_finger_l2, mass 0.03326999; collision mesh filename=package://rby1_description/meshes/rby1m/EE_FINGER.dae; visual mesh filename=package://rby1_description/meshes/rby1m/EE_FINGER.dae
- added link gripper_finger_r1, mass 0.03326999; collision mesh filename=package://rby1_description/meshes/rby1m/EE_FINGER.dae; visual mesh filename=package://rby1_description/meshes/rby1m/EE_FINGER.dae
- added link gripper_finger_r2, mass 0.03326999; collision mesh filename=package://rby1_description/meshes/rby1m/EE_FINGER.dae; visual mesh filename=package://rby1_description/meshes/rby1m/EE_FINGER.dae
- added link gripper_left, mass 0.46704998; collision mesh filename=package://rby1_description/meshes/rby1m/EE_BODY.dae; visual mesh filename=package://rby1_description/meshes/rby1m/EE_BODY.dae
- added link gripper_right, mass 0.46704998; collision mesh filename=package://rby1_description/meshes/rby1m/EE_BODY.dae; visual mesh filename=package://rby1_description/meshes/rby1m/EE_BODY.dae
- link ee_left: mass 0.46704998 -> None; geometry 
- link ee_right: mass 0.46704998 -> None; geometry 
Joints:
- removed joint gripper_finger_l1
- removed joint gripper_finger_l2
- removed joint gripper_finger_r1
- removed joint gripper_finger_r2
- removed joint tool_left
- removed joint tool_right
- added joint ee_left_joint: type fixed, parent link_left_arm_6, child ee_left, origin xyz=0.0 0.0 -0.1261 rpy=0 0.0 0.0, axis 0 0 1
- added joint ee_right_joint: type fixed, parent link_right_arm_6, child ee_right, origin xyz=0.0 0.0 -0.1261 rpy=0 0.0 0.0, axis 0 0 1
- added joint gripper_finger_l1_joint: type prismatic, parent gripper_left, child gripper_finger_l1, origin xyz=0.003 0.0 -0.075 rpy=0.0 0.0 0.0, axis -1 0 0, limit lower=-0.05 upper=0 effort=1000 velocity=0.05
- added joint gripper_finger_l2_joint: type prismatic, parent gripper_left, child gripper_finger_l2, origin xyz=-0.003 0.0 -0.075 rpy=0.0 0.0 3.1415926535, axis 1 0 0, limit lower=0 upper=0.05 effort=1000 velocity=0.05, mimic joint=gripper_finger_l1_joint multiplier=1.0 offset=0.0
- added joint gripper_finger_r1_joint: type prismatic, parent gripper_right, child gripper_finger_r1, origin xyz=0.003 0.0 -0.075 rpy=0.0 0.0 0.0, axis -1 0 0, limit lower=-0.05 upper=0 effort=1000 velocity=0.05
- added joint gripper_finger_r2_joint: type prismatic, parent gripper_right, child gripper_finger_r2, origin xyz=-0.003 0.0 -0.075 rpy=0.0 0.0 3.1415926535, axis 1 0 0, limit lower=0 upper=0.05 effort=1000 velocity=0.05
- added joint gripper_left_joint: type fixed, parent ee_left, child gripper_left, origin xyz=0.0 0.0 0.0 rpy=0 0.0 0.0, axis 0 0 0
- added joint gripper_right_joint: type fixed, parent ee_right, child gripper_right, origin xyz=0.0 0.0 0.0 rpy=0 0.0 0.0, axis 0 0 0

File: rby1_description/urdf/rby1m/model_v1_3.urdf (robot description, URDF)
Before this commit: robot RBY1_M_v1_3, 34 links, 33 joints
Links:
- removed link ee_finger_l1
- removed link ee_finger_l2
- removed link ee_finger_r1
- removed link ee_finger_r2
- added link gripper_finger_l1, mass 0.03326999; collision mesh filename=package://rby1_description/meshes/rby1m/EE_FINGER.dae; visual mesh filename=package://rby1_description/meshes/rby1m/EE_FINGER.dae
- added link gripper_finger_l2, mass 0.03326999; collision mesh filename=package://rby1_description/meshes/rby1m/EE_FINGER.dae; visual mesh filename=package://rby1_description/meshes/rby1m/EE_FINGER.dae
- added link gripper_finger_r1, mass 0.03326999; collision mesh filename=package://rby1_description/meshes/rby1m/EE_FINGER.dae; visual mesh filename=package://rby1_description/meshes/rby1m/EE_FINGER.dae
- added link gripper_finger_r2, mass 0.03326999; collision mesh filename=package://rby1_description/meshes/rby1m/EE_FINGER.dae; visual mesh filename=package://rby1_description/meshes/rby1m/EE_FINGER.dae
- added link gripper_left, mass 0.47470074; collision mesh filename=package://rby1_description/meshes/rby1m/EE_GR_TF.dae; visual mesh filename=package://rby1_description/meshes/rby1m/EE_GR_TF.dae
- added link gripper_right, mass 0.47470074; collision mesh filename=package://rby1_description/meshes/rby1m/EE_GR_TF.dae; visual mesh filename=package://rby1_description/meshes/rby1m/EE_GR_TF.dae
- link ee_left: mass 0.47470074 -> None; geometry 
- link ee_right: mass 0.47470074 -> None; geometry 
Joints:
- removed joint END_left
- removed joint END_right
- removed joint gripper_finger_l1
- removed joint gripper_finger_l2
- removed joint gripper_finger_r1
- removed joint gripper_finger_r2
- added joint ee_left_joint: type fixed, parent link_left_arm_6, child ee_left, origin xyz=0.0 0.0 -0.125 rpy=0 0.0 0.0, axis 0 0 0
- added joint ee_right_joint: type fixed, parent link_right_arm_6, child ee_right, origin xyz=0.0 0.0 -0.125 rpy=0 0.0 0.0, axis 0 0 0
- added joint gripper_finger_l1_joint: type prismatic, parent gripper_left, child gripper_finger_l1, origin xyz=0.0 0.0 0.0 rpy=0 0.0 1.5707963268, axis 1 0 0, limit lower=0.0 upper=0.05 effort=1000 velocity=0.05
- added joint gripper_finger_l2_joint: type prismatic, parent gripper_left, child gripper_finger_l2, origin xyz=0.0 0.0 0.0 rpy=0 0.0 -1.5707963268, axis -1 0 0, limit lower=-0.05 upper=0.0 effort=1000 velocity=0.05, mimic joint=gripper_finger_l1_joint multiplier=1.0 offset=0.0
- added joint gripper_finger_r1_joint: type prismatic, parent gripper_right, child gripper_finger_r1, origin xyz=0.0 0.0 0.0 rpy=0 0.0 1.5707963268, axis 1 0 0, limit lower=0.0 upper=0.05 effort=1000 velocity=0.05
- added joint gripper_finger_r2_joint: type prismatic, parent gripper_right, child gripper_finger_r2, origin xyz=0.0 0.0 0.0 rpy=0 0.0 -1.5707963268, axis -1 0 0, limit lower=-0.05 upper=0.0 effort=1000 velocity=0.05, mimic joint=gripper_finger_r1_joint multiplier=1.0 offset=0.0
- added joint gripper_left_joint: type fixed, parent ee_left, child gripper_left, origin xyz=0.0 0.0 0.0 rpy=0 0.0 0.0, axis 0 0 0
- added joint gripper_right_joint: type fixed, parent ee_right, child gripper_right, origin xyz=0.0 0.0 0.0 rpy=0 0.0 0.0, axis 0 0 0

File: rby1_moveit/rby1_moveit_m_1_2/config/RBY1_M_v1_2.ros2_control.xacro (robot description, xacro)
@@ -3,5 +3,5 @@
     <xacro:macro name="RBY1_M_v1_2_ros2_control" params="name initial_positions_file use_fake_hardware:=true robot_ip:=127.0.0.1:50051 model:=m">
         <xacro:property name="initial_positions" value="${xacro.load_yaml(initial_positions_file)['initial_positions']}"/>
-	<xacro:arg name="robot_ip" default="127.0.0.1:50051" />
+	      <xacro:arg name="robot_ip" default="127.0.0.1:50051" />
         <xacro:arg name="model" default="m" />
         <ros2_control name="${name}" type="system">
@@ -148,4 +148,16 @@
                 </state_interface>
             </joint>
+            <joint name="gripper_finger_r1_joint">
+                <command_interface name="position"/>
+                <state_interface name="position">
+                  <param name="initial_value">${initial_positions['gripper_finger_r1_joint']}</param>
+                </state_interface>
+            </joint>
+            <joint name="gripper_finger_l1_joint">
+                <command_interface name="position"/>
+                <state_interface name="position">
+                  <param name="initial_value">${initial_positions['gripper_finger_l1_joint']}</param>
+                </state_interface>
+            </joint>
         </ros2_control>
     </xacro:macro>
